File: dad_bob_kicad/dad_bob_diff.sch (KiCad schematic (older format))
At the start: 70 parts

Commit message: Added pcbNew files, block layouts complete
Parts:
- removed C?: ~, symbol Device:C
- removed R?: ~, symbol Device:R
- C22, C23, C24, C25, C26, C27, C28, C29, C30, C32, C33, C34, C36, C37, C38, C39, C40, C41, C42, C43, C44, C45, C46, C47, C48, C49, C50, C51, C52, C53, C54, C55, C56: renamed from C?; footprint (none) -> Capacitor_SMD:C_0805_2012Metric_Pad1.15x1.40mm_HandSolder
- C31, C35: renamed from C?; footprint (none) -> Capacitor_SMD:C_Trimmer_Voltronics_JQ
- FB1, FB2, FB3: renamed from FB?; footprint (none) -> Ferrite_THT:LairdTech_28C0236-0JW-10
- R17, R18, R19, R20, R21, R22, R23, R24, R25, R26, R27, R28, R29, R30, R31, R32, R33, R34, R35, R36, R37, R38, R39: renamed from R?; footprint (none) -> Resistor_SMD:R_0805_2012Metric_Pad1.15x1.40mm_HandSolder
- U4: renamed from U?; symbol LM7301IMX_NOPB:LM7301 -> 00_kyuditsky_kicad:LM7301
- gave numbers to parts that had none: 4
Connections:
- net VCC: no longer C27.2, C36.2, C37.2, C46.1, C47.1, C48.1, C49.1, C51.1, C52.1, C53.1, C54.1, C55.1, C56.1, FB3.1, R39.2, U2.4 (V-), U3.2 (V-), U4.4 (V-)
- new net greg: C27.2, C36.2, C37.2, C46.1, C47.1, C48.1, C49.1, C51.1, C52.1, C53.1, C54.1, C55.1, C56.1, FB3.1, R39.2, U2.4 (V-), U3.2 (V-), U4.4 (V-)

Commit message: changed some layout, realized it needs some rework, but versioning for posterity
Parts:
- U4: value LTC6269 -> LM7301
Connections:
- net V- is gone; now on net GND: C50.1, FB3.2, Q3.1 (G)
- net GND: no longer C22.1, C28.1, C36.1, C37.1, C44.2, C45.2, C47.2, C48.2, C54.2, C55.2, C56.2, FB2.1, J11.2, J11.3, J11.4, J11.5, R25.1, R29.1
- new net GNDREF: C22.1, C28.1, C36.1, C37.1, C44.2, C45.2, C47.2, C48.2, C54.2, C55.2, C56.2, FB2.1, J11.2, J11.3, J11.4, J11.5, R25.1, R29.1
Changed lines of the file:
@@
 	0    1    1    0
-$EndComp
-$Comp
-L power:GND #PWR?
-U 1 1 624AA0BB
-P 5450 3650
-AR Path="/624AA0BB" Ref="#PWR?"  Part="1"
-AR Path="/624874CF/624AA0BB" Ref="#PWR015"  Part="1"
-F 0 "#PWR015" H 5450 3400 50  0001 C CNN
-F 1 "GND" V 5455 3522 50  0000 R CNN
-F 2 "" H 5450 3650 50  0001 C CNN
-F 3 "" H 5450 3650 50  0001 C CNN
-	1    5450 3650
-	1    0    0    -1
 $EndComp
 Connection ~ 3500 2900
@@
 	1    6750 4350
 	0    1    1    0
-$EndComp
-$Comp
-L power:GND #PWR?
-U 1 1 624C45F2
-P 7050 3700
-AR Path="/624C45F2" Ref="#PWR?"  Part="1"
-AR Path="/624874CF/624C45F2" Ref="#PWR016"  Part="1"
-F 0 "#PWR016" H 7050 3450 50  0001 C CNN
-F 1 "GND" V 7055 3572 50  0000 R CNN
-F 2 "" H 7050 3700 50  0001 C CNN
-F 3 "" H 7050 3700 50  0001 C CNN
-	1    7050 3700
-	1    0    0    -1
 $EndComp
 $Comp
@@
 Wire Wire Line
 	8050 2450 8050 2750
-$Comp
-L power:GND #PWR?
-U 1 1 6252E790
-P 8200 2850
-AR Path="/6252E790" Ref="#PWR?"  Part="1"
-AR Path="/624874CF/6252E790" Ref="#PWR014"  Part="1"
-F 0 "#PWR014" H 8200 2600 50  0001 C CNN
-F 1 "GND" V 8205 2722 50  0000 R CNN
-F 2 "" H 8200 2850 50  0001 C CNN
-F 3 "" H 8200 2850 50  0001 C CNN
-	1    8200 2850
-	1    0    0    -1
-$EndComp
 Wire Wire Line
 	8050 2750 8200 2750
@@
 Wire Wire Line
 	8450 3850 8450 4150
-$Comp
-L power:GND #PWR?
-U 1 1 6253B673
-P 8550 4250
-AR Path="/6253B673" Ref="#PWR?"  Part="1"
-AR Path="/624874CF/6253B673" Ref="#PWR017"  Part="1"
-F 0 "#PWR017" H 8550 4000 50  0001 C CNN
-F 1 "GND" V 8555 4122 50  0000 R CNN
-F 2 "" H 8550 4250 50  0001 C CNN
-F 3 "" H 8550 4250 50  0001 C CNN
-	1    8550 4250
-	1    0    0    -1
-$EndComp
 Wire Wire Line
 	8550 4150 8450 4150
@@
 Wire Wire Line
 	10300 5800 10300 5750
-$Comp
-L power:GND #PWR?
-U 1 1 6259C3AA
-P 9500 6100
-AR Path="/6259C3AA" Ref="#PWR?"  Part="1"
-AR Path="/624874CF/6259C3AA" Ref="#PWR018"  Part="1"
-F 0 "#PWR018" H 9500 5850 50  0001 C CNN
-F 1 "GND" V 9505 5972 50  0000 R CNN
-F 2 "" H 9500 6100 50  0001 C CNN
-F 3 "" H 9500 6100 50  0001 C CNN
-	1    9500 6100
-	1    0    0    -1
-$EndComp
 Wire Wire Line
 	9500 6100 9500 5900
@@
 P 4450 6800
 F 0 "U4" H 4600 6900 50  0000 L CNN
-F 1 "LTC6269" H 4500 7000 50  0000 L CNN
+F 1 "LM7301" H 4500 7000 50  0000 L CNN
 F 2 "LTC6269:SOP65P490X110-9N" H 4450 6800 50  0001 C CNN
 F 3 "https://www.analog.com/media/en/technical-documentation/data-sheets/62689f.pdf" H 4450 6800 50  0001 C CNN
@@
 	1    0    0    1
 $EndComp
-Text GLabel 1300 7200 0    50   Input ~ 0
-V-
 $Comp
 L Device:C C?
@@
 	-1   0    0    1
 $EndComp
-$Comp
-L power:GND #PWR?
-U 1 1 6241649B
-P 6500 6850
-AR Path="/6241649B" Ref="#PWR?"  Part="1"
-AR Path="/624874CF/6241649B" Ref="#PWR019"  Part="1"
-F 0 "#PWR019" H 6500 6600 50  0001 C CNN
-F 1 "GND" V 6505 6722 50  0000 R CNN
-F 2 "" H 6500 6850 50  0001 C CNN
-F 3 "" H 6500 6850 50  0001 C CNN
-	1    6500 6850
-	1    0    0    -1
-$EndComp
 Wire Wire Line
 	4000 6900 4050 6900
@@
 Wire Wire Line
 	5250 6800 5450 6800
-Wire Wire Line
-	6500 6800 6500 6850
 Connection ~ 5450 6800
 Wire Wire Line
@@
 Wire Wire Line
 	1700 6750 1700 7200
-Wire Wire Line
-	1700 7200 1300 7200
 Wire Wire Line
 	1700 7200 2050 7200
@@
 	3600 7350 3700 7350
 Connection ~ 3700 7350
+Wire Wire Line
+	1300 7200 1700 7200
+$Comp
+L power:GNDREF #PWR020
+U 1 1 626A2E1B
+P 6500 6950
+F 0 "#PWR020" H 6500 6700 50  0001 C CNN
+F 1 "GNDREF" H 6505 6777 50  0000 C CNN
+F 2 "" H 6500 6950 50  0001 C CNN
+F 3 "" H 6500 6950 50  0001 C CNN
+	1    6500 6950
+	1    0    0    -1
+$EndComp
+Wire Wire Line
+	6500 6800 6500 6950
+$Comp
+L power:GNDREF #PWR019
+U 1 1 626AD60A
+P 9500 6100
+F 0 "#PWR019" H 9500 5850 50  0001 C CNN
+F 1 "GNDREF" H 9505 5927 50  0000 C CNN
+F 2 "" H 9500 6100 50  0001 C CNN
+F 3 "" H 9500 6100 50  0001 C CNN
+	1    9500 6100
+	1    0    0    -1
+$EndComp
+$Comp
+L power:GNDREF #PWR018
+U 1 1 626AE74B
+P 8550 4250
+F 0 "#PWR018" H 8550 4000 50  0001 C CNN
+F 1 "GNDREF" H 8555 4077 50  0000 C CNN
+F 2 "" H 8550 4250 50  0001 C CNN
+F 3 "" H 8550 4250 50  0001 C CNN
+	1    8550 4250
+	1    0    0    -1
+$EndComp
+$Comp
+L power:GNDREF #PWR015
+U 1 1 626B0246
+P 8200 2850
+F 0 "#PWR015" H 8200 2600 50  0001 C CNN
+F 1 "GNDREF" H 8205 2677 50  0000 C CNN
+F 2 "" H 8200 2850 50  0001 C CNN
+F 3 "" H 8200 2850 50  0001 C CNN
+	1    8200 2850
+	1    0    0    -1
+$EndComp
+$Comp
+L power:GNDREF #PWR016
+U 1 1 626B06B3
+P 5450 3650
+F 0 "#PWR016" H 5450 3400 50  0001 C CNN
+F 1 "GNDREF" H 5455 3477 50  0000 C CNN
+F 2 "" H 5450 3650 50  0001 C CNN
+F 3 "" H 5450 3650 50  0001 C CNN
+	1    5450 3650
+	1    0    0    -1
+$EndComp
+$Comp
+L power:GNDREF #PWR017
+U 1 1 626B15D9
+P 7050 3750
+F 0 "#PWR017" H 7050 3500 50  0001 C CNN
+F 1 "GNDREF" H 7055 3577 50  0000 C CNN
+F 2 "" H 7050 3750 50  0001 C CNN
+F 3 "" H 7050 3750 50  0001 C CNN
+	1    7050 3750
+	1    0    0    -1
+$EndComp
+Wire Wire Line
+	7050 3750 7050 3700
+$Comp
+L power:GND #PWR0101
+U 1 1 627C0A0D
+P 1300 7200
+F 0 "#PWR0101" H 1300 6950 50  0001 C CNN
+F 1 "GND" V 1305 7072 50  0000 R CNN
+F 2 "" H 1300 7200 50  0001 C CNN
+F 3 "" H 1300 7200 50  0001 C CNN
+	1    1300 7200
+	0    1    1    0
+$EndComp
 $EndSCHEMATC
