File: dad_bod_kicad/dad_bod_diff.kicad_sch (KiCad schematic)
At the start: 66 parts

Commit message: Routed PCB, layout needs rework, forked to dad_bod
Parts:
- C22, C27, C28, C32, C36, C37, C42, C43, C44, C45, C46, C47, C48, C49, C50, C51, C52, C53, C54, C55, C56: renamed from C?; value (none) -> ~; footprint (none) -> Capacitor_SMD:C_0805_2012Metric_Pad1.15x1.40mm_HandSolder
- C23, C24, C25, C26, C38, C39, C40, C41: renamed from C?; value (none) -> 4pf; footprint (none) -> Capacitor_SMD:C_0805_2012Metric_Pad1.15x1.40mm_HandSolder
- C29, C30, C33, C34: renamed from C?; value (none) -> 350pF; footprint (none) -> Capacitor_SMD:C_0805_2012Metric_Pad1.15x1.40mm_HandSolder
- C31, C35: value (none) -> CTRIM; footprint (none) -> Capacitor_SMD:C_Trimmer_Voltronics_JQ
- FB1, FB2, FB3: value (none) -> Ferrite_Bead; footprint (none) -> Ferrite_THT:LairdTech_28C0236-0JW-10
- J11: renamed from J?; value (none) -> BNC5-J-P-GN-RA-BH2D; footprint (none) -> BNC5-J-P-GN-RA-BH2D_kicad:BNC5JPGNRABH2D
- Q3: value (none) -> AO3401A; footprint (none) -> Package_TO_SOT_SMD:SOT-23
- R17, R18, R23, R26, R27, R29, R34, R35, R36, R37, R38, R39: renamed from R?; value (none) -> ~; footprint (none) -> Resistor_SMD:R_0805_2012Metric_Pad1.15x1.40mm_HandSolder
- R19, R20, R21, R22, R30, R31, R32, R33: renamed from R?; value (none) -> 1M; footprint (none) -> Resistor_SMD:R_0805_2012Metric_Pad1.15x1.40mm_HandSolder
- R24, R28: renamed from R?; value (none) -> 50k; footprint (none) -> Resistor_SMD:R_0805_2012Metric_Pad1.15x1.40mm_HandSolder
- R25: renamed from R?; value (none) -> DNP; footprint (none) -> Resistor_SMD:R_0805_2012Metric_Pad1.15x1.40mm_HandSolder
- U2: value (none) -> LTC6269; footprint (none) -> LTC6269:SOP65P490X110-9N
- U3: value (none) -> LTC6268; footprint (none) -> LTC6268IS6-10#TRMPBF:SOT95P280X100-6N
- U4: value (none) -> LM7301; footprint (none) -> LTC6269:SOP65P490X110-9N
