File: dad_bod_kicad/dad_bod.kicad_sch (KiCad schematic)
At the start: 67 parts, among them J1 Conn_01x01, J10 Conn_01x03_Male, J12 USB4085-GF-A_REVA4, J13 Conn_01x03_Male, J14 Conn_01x03_Male, J2 Conn_01x01, J3 Conn_01x01, J4 Conn_01x01, J5 Conn_01x03_Male, J6 Conn_02x15_Odd_Even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

Commit message: changed some routing/footprints after component selection
Parts:
- C5, C6: footprint Capacitor_SMD:C_0805_2012Metric_Pad1.15x1.40mm_HandSolder -> kyuditsky_kicad:EEE1AA220WR
- D1: value SMCJ9.0CA -> SMCJ918.0CA
Other:
- note added: "Made C2 0805"
- note added: "switched to: SMCJ18.0CA"
- note removed: "Made C2 0806"
- note removed: "switched to: SMCJ9.0CA"
Changed lines of the file:
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@@
     (stroke (width 0) (type default) (color 0 0 0 0))
   )
-  (text "Made C2 0806" (at 193.04 34.29 0)
+  (text "Made C2 0805" (at 193.04 34.29 0)
     (effects (font (size 1.27 1.27)) (justify left bottom))
   )
@@
     (effects (font (size 1.27 1.27)) (justify right bottom))
   )
-  (text "switched to: SMCJ9.0CA" (at 163.83 43.18 0)
+  (text "switched to: SMCJ18.0CA" (at 163.83 43.18 0)
     (effects (font (size 1.27 1.27)) (justify left bottom))
   )
@@
     )
   )
-  (global_label "DIVout1+" (shape output) (at 90.17 185.42 0) (fields_autoplaced)
-    (effects (font (size 1.27 1.27)) (justify left))
-    (property "Intersheet References" "${INTERSHEET_REFS}" (id 0) (at 0 0 0)
-      (effects (font (size 1.27 1.27)) hide)
-    )
-  )
   (global_label "scope1-" (shape input) (at 257.81 72.39 0) (fields_autoplaced)
     (effects (font (size 1.27 1.27)) (justify left))
@@
     )
   )
-  (global_label "DIVin1+" (shape input) (at 87.63 185.42 180) (fields_autoplaced)
-    (effects (font (size 1.27 1.27)) (justify right))
-    (property "Intersheet References" "${INTERSHEET_REFS}" (id 0) (at 0 0 0)
-      (effects (font (size 1.27 1.27)) hide)
-    )
-  )
   (global_label "15" (shape bidirectional) (at 240.03 59.69 180) (fields_autoplaced)
     (effects (font (size 1.27 1.27)) (justify right))
@@
     )
   )
-  (global_label "DIVin1-" (shape input) (at 87.63 190.5 180) (fields_autoplaced)
-    (effects (font (size 1.27 1.27)) (justify right))
-    (property "Intersheet References" "${INTERSHEET_REFS}" (id 0) (at 0 0 0)
-      (effects (font (size 1.27 1.27)) hide)
-    )
-  )
   (global_label "2" (shape bidirectional) (at 257.81 46.99 0) (fields_autoplaced)
     (effects (font (size 1.27 1.27)) (justify left))
@@
     (property "Intersheet References" "${INTERSHEET_REFS}" (id 0) (at 0 99.06 0)
       (effects (font (size 1.27 1.27)) (justify left) hide)
-    )
-  )
-  (global_label "DIVout1-" (shape output) (at 90.17 190.5 0) (fields_autoplaced)
-    (effects (font (size 1.27 1.27)) (justify left))
-    (property "Intersheet References" "${INTERSHEET_REFS}" (id 0) (at 0 0 0)
-      (effects (font (size 1.27 1.27)) hide)
     )
   )
@@
     (property "Reference" "C5" (id 0) (at 115.57 62.103 90))
     (property "Value" "CP" (id 1) (at 115.57 64.4144 90))
-    (property "Footprint" "Capacitor_SMD:C_0805_2012Metric_Pad1.15x1.40mm_HandSolder" (id 2) (at 111.76 69.5452 0)
+    (property "Footprint" "kyuditsky_kicad:EEE1AA220WR" (id 2) (at 111.76 69.5452 0)
       (effects (font (size 1.27 1.27)) hide)
     )
@@
     (property "Reference" "C6" (id 0) (at 181.61 62.103 90))
     (property "Value" "CP" (id 1) (at 181.61 64.4144 90))
-    (property "Footprint" "Capacitor_SMD:C_0805_2012Metric_Pad1.15x1.40mm_HandSolder" (id 2) (at 177.8 69.5452 0)
+    (property "Footprint" "kyuditsky_kicad:EEE1AA220WR" (id 2) (at 177.8 69.5452 0)
       (effects (font (size 1.27 1.27)) hide)
     )
@@
       (effects (font (size 1.27 1.27)) (justify left))
     )
-    (property "Value" "SMCJ9.0CA" (id 1) (at 175.26 25.4 0)
+    (property "Value" "SMCJ918.0CA" (id 1) (at 175.26 25.4 0)
       (effects (font (size 1.27 1.27)) (justify left))
     )
@@
   (symbol (lib_id "Device:R") (at 203.2 130.81 90) (unit 1)
     (in_bom yes) (on_board yes)
-    (property "Reference" "R40" (id 0) (at 199.39 128.27 90))
+    (property "Reference" "R40" (id 0) (at 198.755 128.27 90))
     (property "Value" "5.1k" (id 1) (at 203.2 128.27 90))
     (property "Footprint" "Resistor_SMD:R_0805_2012Metric_Pad1.15x1.40mm_HandSolder" (id 2) (at 203.2 132.588 90)
@@
     )
     (path "/00000000-0000-0000-0000-00006210de69"
-      (reference "C5") (unit 1) (value "CP") (footprint "Capacitor_SMD:C_0805_2012Metric_Pad1.15x1.40mm_HandSolder")
+      (reference "C5") (unit 1) (value "CP") (footprint "kyuditsky_kicad:EEE1AA220WR")
     )
     (path "/00000000-0000-0000-0000-000062249300"
-      (reference "C6") (unit 1) (value "CP") (footprint "Capacitor_SMD:C_0805_2012Metric_Pad1.15x1.40mm_HandSolder")
+      (reference "C6") (unit 1) (value "CP") (footprint "kyuditsky_kicad:EEE1AA220WR")
     )
     (path "/00000000-0000-0000-0000-000062298c93"
@@
     )
     (path "/00000000-0000-0000-0000-0000623e98ab"
-      (reference "D1") (unit 1) (value "SMCJ9.0CA") (footprint "SMCJ5:DIONM7959X262N")
+      (reference "D1") (unit 1) (value "SMCJ918.0CA") (footprint "SMCJ5:DIONM7959X262N")
     )
     (path "/00000000-0000-0000-0000-0000620ff5ac"
@@
       (reference "D6") (unit 1) (value "SMCJ5.0A") (footprint "kyuditsky_kicad_fp:littlefuseTVS")
     )
+    (path "/00000000-0000-0000-0000-0000624874cf/ec978c9e-3baa-4273-9c24-b663927a950a"
+      (reference "D7") (unit 1) (value "BAV199-TP") (footprint "kyuditsky_kicad:bav199_tp_SOT95P237X125-3N")
+    )
+    (path "/00000000-0000-0000-0000-0000624874cf/edb8a1e7-6a49-4f5e-b9d9-de960c16dd4e"
+      (reference "D8") (unit 1) (value "BAV199-TP") (footprint "kyuditsky_kicad:bav199_tp_SOT95P237X125-3N")
+    )
     (path "/00000000-0000-0000-0000-000062690ea2"

Commit message: swapped div1 & div 2 inputs, bnc in can be routed as plc out
Parts:
- removed E1: SPARK_GAP, symbol dad_bob-rescue:SPARK_GAP-Device
- removed J14: Conn_01x03_Male, Connector_PinHeader_2.54mm:PinHeader_1x03_P2.54mm_Vertical, symbol Connector:Conn_01x03_Male
Connections:
- net PLCout- is gone; now on net BNCin-: C2.1, D1.2, K1.8, T1.4 (GATE_1)
- net CV6: now also R3.1; no longer J13.1 (Pin_1)
- net CV7: now also R4.1
- net DIVin1+: now also C7.2, J10.1 (Pin_1); no longer C4.2, J8.1 (Pin_1), T1.1 (DRIVE_1), U1.2
- net DIVin1-: now also J3.1 (Pin_1), R5.1; no longer C1.1, J1.1 (Pin_1), R2.1, RV1.2
- net DIVin2+: now also C1.1, J1.1 (Pin_1), R2.1, RV1.2; no longer J3.1 (Pin_1), R5.1
- net DIVin2-: now also C4.2, J8.1 (Pin_1), T1.1 (DRIVE_1), U1.2; no longer C7.2, J10.1 (Pin_1)
- net DIVout1+: now also K2.8; no longer K1.3
- net DIVout1-: now also K2.5; no longer K1.10
- net DIVout2+: now also K1.3; no longer K2.5
- net DIVout2-: now also K1.10; no longer K2.8
- net PLCout+: now also J13.1 (Pin_1)
- net V+: no longer J13.3 (Pin_3)
- net bnc_imp+: now reaches J5.2 (Pin_2), R1.2
- net bnc_imp+: now also J13.3 (Pin_3); no longer J7.1
- net at J13.2 (Pin_2): now also J7.1; no longer R3.1
Other:
- moved on the sheet: C3, J5, J7, R1

Commit message: touch ups & final review
Connections:
- net DIVout1+: now also K2.5; no longer K2.8
- net DIVout1-: now also K2.8; no longer K2.5
Changed lines of the file:
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@@
     )
   )
-  (global_label "DIVout1+" (shape input) (at 210.82 68.58 90) (fields_autoplaced)
+  (global_label "DIVout1+" (shape input) (at 200.66 68.58 90) (fields_autoplaced)
     (effects (font (size 1.27 1.27)) (justify left))
-    (property "Intersheet References" "${INTERSHEET_REFS}" (id 0) (at 81.28 0 0)
+    (property "Intersheet References" "${INTERSHEET_REFS}" (id 0) (at 71.12 0 0)
       (effects (font (size 1.27 1.27)) hide)
     )
@@
     )
   )
-  (global_label "DIVout1-" (shape input) (at 200.66 68.58 90) (fields_autoplaced)
+  (global_label "DIVout1-" (shape input) (at 210.82 68.58 90) (fields_autoplaced)
     (effects (font (size 1.27 1.27)) (justify left))
-    (property "Intersheet References" "${INTERSHEET_REFS}" (id 0) (at 60.96 0 0)
+    (property "Intersheet References" "${INTERSHEET_REFS}" (id 0) (at 71.12 0 0)
       (effects (font (size 1.27 1.27)) hide)
     )
